File: Hardware/0. Project/Soil Moisture Meter (IoT Device).brd (EAGLE design)
At the start: 30 x 200 mm, 22 parts, among them J1 ICSP, Q1 32.768 kHz, U1 MSP430FR4133

Commit message: Changed folder structure
Parts:
- R6, R7: value 10k -> 0R
Changed lines of the file:
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@@
 <drawing>
 <settings>
-<setting alwaysvectorfont="yes"/>
+<setting alwaysvectorfont="no"/>
 <setting verticaltext="up"/>
 </settings>
@@
 <attribute name="VALUE" x="17.336" y="167.593" size="1.27" layer="27" align="center" display="off"/>
 </element>
-<element name="R6" library="rcl" library_urn="urn:adsk.eagle:library:334" package="R0603" package3d_urn="urn:adsk.eagle:package:23555/3" value="10k" x="25" y="146.75" smashed="yes" rot="R90">
+<element name="R6" library="rcl" library_urn="urn:adsk.eagle:library:334" package="R0603" package3d_urn="urn:adsk.eagle:package:23555/3" value="0R" x="25" y="146.75" smashed="yes" rot="R90">
 <attribute name="NAME" x="24.365" y="146.115" size="1.27" layer="25" rot="R90" display="off"/>
 <attribute name="SPICEPREFIX" value="R" x="25" y="146.75" size="1.778" layer="27" rot="R90" display="off"/>
 <attribute name="VALUE" x="26.905" y="146.115" size="1.27" layer="27" rot="R90" display="off"/>
 </element>
-<element name="R7" library="rcl" library_urn="urn:adsk.eagle:library:334" package="R0603" package3d_urn="urn:adsk.eagle:package:23555/3" value="10k" x="5" y="147" smashed="yes" rot="R270">
+<element name="R7" library="rcl" library_urn="urn:adsk.eagle:library:334" package="R0603" package3d_urn="urn:adsk.eagle:package:23555/3" value="0R" x="5" y="147" smashed="yes" rot="R270">
 <attribute name="NAME" x="5.635" y="147.635" size="1.27" layer="25" rot="R270" display="off"/>
 <attribute name="SPICEPREFIX" value="R" x="5" y="147" size="1.778" layer="27" rot="R270" display="off"/>
